File: pcb/can-module/totem-pole.kicad_sch (KiCad schematic)
At the start: 6 parts, among them Q4 2N7002, Q5 AO3401A, Q6 2N7002

Commit message: Board layout
Parts:
- renumbered Q6 to Q10, Q5 to Q11, Q4 to Q12, R9 to R20, R8 to R21, R7 to R24
Changed lines of the file:
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@@
 		(on_board yes)
 		(dnp no)
-		(property "Reference" "R9"
+		(property "Reference" "R20"
 			(at 129.54 101.6 0)
 			(effects
@@
 			(project "can-module"
 				(path "/8c0b3d8b-46d3-4173-ab1e-a61765f77d61/09a5a7b6-fe3e-4eb4-9cde-bb28b08e6e92"
-					(reference "R24")
+					(reference "R8")
 					(unit 1)
 				)
@@
 				)
 				(path "/8c0b3d8b-46d3-4173-ab1e-a61765f77d61/b63ae371-0413-4524-b027-6b09efc1ff94"
-					(reference "R9")
+					(reference "R20")
 					(unit 1)
 				)
 				(path "/8c0b3d8b-46d3-4173-ab1e-a61765f77d61/b9c0ee24-df58-437e-92df-5944137f34d2"
-					(reference "R20")
+					(reference "R12")
 					(unit 1)
 				)
@@
 		(on_board yes)
 		(dnp no)
-		(property "Reference" "R8"
+		(property "Reference" "R21"
 			(at 125.73 73.66 0)
 			(effects
@@
 			(project "can-module"
 				(path "/8c0b3d8b-46d3-4173-ab1e-a61765f77d61/09a5a7b6-fe3e-4eb4-9cde-bb28b08e6e92"
-					(reference "R23")
+					(reference "R10")
 					(unit 1)
 				)
 				(path "/8c0b3d8b-46d3-4173-ab1e-a61765f77d61/95cdb4ae-2820-47a5-b7b5-18525147b410"
-					(reference "R15")
+					(reference "R18")
 					(unit 1)
 				)
 				(path "/8c0b3d8b-46d3-4173-ab1e-a61765f77d61/b63ae371-0413-4524-b027-6b09efc1ff94"
-					(reference "R8")
+					(reference "R21")
 					(unit 1)
 				)
 				(path "/8c0b3d8b-46d3-4173-ab1e-a61765f77d61/b9c0ee24-df58-437e-92df-5944137f34d2"
-					(reference "R19")
+					(reference "R13")
 					(unit 1)
 				)
@@
 		(on_board yes)
 		(dnp no)
-		(property "Reference" "Q4"
+		(property "Reference" "Q12"
 			(at 114.3 91.44 0)
 			(effects
@@
 			(project "can-module"
 				(path "/8c0b3d8b-46d3-4173-ab1e-a61765f77d61/09a5a7b6-fe3e-4eb4-9cde-bb28b08e6e92"
-					(reference "Q13")
+					(reference "Q3")
 					(unit 1)
 				)
 				(path "/8c0b3d8b-46d3-4173-ab1e-a61765f77d61/95cdb4ae-2820-47a5-b7b5-18525147b410"
-					(reference "Q7")
+					(reference "Q9")
 					(unit 1)
 				)
 				(path "/8c0b3d8b-46d3-4173-ab1e-a61765f77d61/b63ae371-0413-4524-b027-6b09efc1ff94"
-					(reference "Q4")
+					(reference "Q12")
 					(unit 1)
 				)
 				(path "/8c0b3d8b-46d3-4173-ab1e-a61765f77d61/b9c0ee24-df58-437e-92df-5944137f34d2"
-					(reference "Q10")
+					(reference "Q5")
 					(unit 1)
 				)
@@
 		(on_board yes)
 		(dnp no)
-		(property "Reference" "Q6"
+		(property "Reference" "Q10"
 			(at 138.43 101.6 0)
 			(effects
@@
 			(project "can-module"
 				(path "/8c0b3d8b-46d3-4173-ab1e-a61765f77d61/09a5a7b6-fe3e-4eb4-9cde-bb28b08e6e92"
-					(reference "Q15")
+					(reference "Q1")
 					(unit 1)
 				)
 				(path "/8c0b3d8b-46d3-4173-ab1e-a61765f77d61/95cdb4ae-2820-47a5-b7b5-18525147b410"
-					(reference "Q9")
+					(reference "Q7")
 					(unit 1)
 				)
 				(path "/8c0b3d8b-46d3-4173-ab1e-a61765f77d61/b63ae371-0413-4524-b027-6b09efc1ff94"
-					(reference "Q6")
+					(reference "Q10")
 					(unit 1)
 				)
 				(path "/8c0b3d8b-46d3-4173-ab1e-a61765f77d61/b9c0ee24-df58-437e-92df-5944137f34d2"
-					(reference "Q12")
+					(reference "Q4")
 					(unit 1)
 				)
@@
 		(on_board yes)
 		(dnp no)
-		(property "Reference" "R7"
+		(property "Reference" "R24"
 			(at 96.266 87.63 0)
 			(effects
@@
 			(project "can-module"
 				(path "/8c0b3d8b-46d3-4173-ab1e-a61765f77d61/09a5a7b6-fe3e-4eb4-9cde-bb28b08e6e92"
-					(reference "R21")
+					(reference "R11")
 					(unit 1)
 				)
 				(path "/8c0b3d8b-46d3-4173-ab1e-a61765f77d61/95cdb4ae-2820-47a5-b7b5-18525147b410"
-					(reference "R10")
+					(reference "R19")
 					(unit 1)
 				)
 				(path "/8c0b3d8b-46d3-4173-ab1e-a61765f77d61/b63ae371-0413-4524-b027-6b09efc1ff94"
-					(reference "R7")
+					(reference "R24")
 					(unit 1)
 				)
 				(path "/8c0b3d8b-46d3-4173-ab1e-a61765f77d61/b9c0ee24-df58-437e-92df-5944137f34d2"
-					(reference "R17")
+					(reference "R15")
 					(unit 1)
 				)
@@
 		(on_board yes)
 		(dnp no)
-		(property "Reference" "Q5"
+		(property "Reference" "Q11"
 			(at 138.43 78.74 0)
 			(effects
@@
 			(project "can-module"
 				(path "/8c0b3d8b-46d3-4173-ab1e-a61765f77d61/09a5a7b6-fe3e-4eb4-9cde-bb28b08e6e92"
-					(reference "Q14")
+					(reference "Q2")
 					(unit 1)
 				)
@@
 				)
 				(path "/8c0b3d8b-46d3-4173-ab1e-a61765f77d61/b63ae371-0413-4524-b027-6b09efc1ff94"
-					(reference "Q5")
+					(reference "Q11")
 					(unit 1)
 				)
 				(path "/8c0b3d8b-46d3-4173-ab1e-a61765f77d61/b9c0ee24-df58-437e-92df-5944137f34d2"
-					(reference "Q11")
-					(unit 1)
-				)
+					(reference "Q6")
+					(unit 1)
+				)
